Commit message: feat: add motor+gearbox pairs to all 7 hand joints
- Rework hand_7dof.urdf: each joint now has motor_link + gearbox_link
  chain: parent_link -> motor_link -> gearbox_link -> joint -> child_link
- Realistic specs per joint (Maxon EC motors + GP planetary gearheads):
  gear ratios 6:1 to 12:1, masses 40-200 g, diameters 20-50 mm
- Computed solid-cylinder inertia for every motor/gearbox link
- Gazebo materials: DarkGray (motor) / Black (gearbox)
- Original joint pose/axis/limits/dynamics preserved, re-parented to gearbox_link
- Each joint gets <transmission> with mechanicalReduction for ros2_control
- New: hand_7dof_gazebo.xacro (14 JointPositionController plugins)
- New: config/ros2_control_hand.yaml motor/gearbox parameters block
- New: scripts/add_motors.py (SDF motor+gearbox injector)
- New: full.sdf (29 links, 28 joints) and hand_world.sdf (Gazebo world)
- Updated README with motor/gearbox specs table and kinematic chain docs

File: freecad_hand_7dof/urdf/fetch_7dof_with_hand.urdf (robot description, URDF)
Before this commit: robot fetch_7dof, 17 links, 16 joints
Links:
- added link finger_L_gearbox_link, mass 0.060; collision cylinder length=0.025 radius=0.014; visual cylinder length=0.025 radius=0.014
- added link finger_L_motor_link, mass 0.040; collision cylinder length=0.030 radius=0.010; visual cylinder length=0.030 radius=0.010
- added link finger_R_gearbox_link, mass 0.060; collision cylinder length=0.025 radius=0.014; visual cylinder length=0.025 radius=0.014
- added link finger_R_motor_link, mass 0.040; collision cylinder length=0.030 radius=0.010; visual cylinder length=0.030 radius=0.010
- added link hand_pitch_gearbox_link, mass 0.200; collision cylinder length=0.040 radius=0.025; visual cylinder length=0.040 radius=0.025
- added link hand_pitch_motor_link, mass 0.150; collision cylinder length=0.030 radius=0.0225; visual cylinder length=0.030 radius=0.0225
- added link hand_roll_gearbox_link, mass 0.120; collision cylinder length=0.035 radius=0.019; visual cylinder length=0.035 radius=0.019
- added link hand_roll_motor_link, mass 0.080; collision cylinder length=0.040 radius=0.016; visual cylinder length=0.040 radius=0.016
- added link hand_yaw_gearbox_link, mass 0.200; collision cylinder length=0.040 radius=0.025; visual cylinder length=0.040 radius=0.025
- added link hand_yaw_motor_link, mass 0.150; collision cylinder length=0.030 radius=0.0225; visual cylinder length=0.030 radius=0.0225
- added link knuckle_spread_L_gearbox_link, mass 0.080; collision cylinder length=0.025 radius=0.014; visual cylinder length=0.025 radius=0.014
- added link knuckle_spread_L_motor_link, mass 0.050; collision cylinder length=0.030 radius=0.011; visual cylinder length=0.030 radius=0.011
- added link knuckle_spread_R_gearbox_link, mass 0.080; collision cylinder length=0.025 radius=0.014; visual cylinder length=0.025 radius=0.014
- added link knuckle_spread_R_motor_link, mass 0.050; collision cylinder length=0.030 radius=0.011; visual cylinder length=0.030 radius=0.011
Joints:
- added joint finger_L_gearbox_fixed: type fixed, parent finger_L_motor_link, child finger_L_gearbox_link, origin xyz=0 0 0
- added joint finger_L_motor_fixed: type fixed, parent hand_knuckle_l_link, child finger_L_motor_link, origin xyz=0.012 -0.005 0.015
- added joint finger_R_gearbox_fixed: type fixed, parent finger_R_motor_link, child finger_R_gearbox_link, origin xyz=0 0 0
- added joint finger_R_motor_fixed: type fixed, parent hand_knuckle_r_link, child finger_R_motor_link, origin xyz=0.012 0.005 0.015
- added joint hand_pitch_gearbox_fixed: type fixed, parent hand_pitch_motor_link, child hand_pitch_gearbox_link, origin xyz=0 0 0
- added joint hand_pitch_motor_fixed: type fixed, parent hand_yaw_link, child hand_pitch_motor_link, origin xyz=0.025 0 0
- added joint hand_roll_gearbox_fixed: type fixed, parent hand_roll_motor_link, child hand_roll_gearbox_link, origin xyz=0 0 0
- added joint hand_roll_motor_fixed: type fixed, parent hand_pitch_link, child hand_roll_motor_link, origin xyz=0.025 0 0
- added joint hand_yaw_gearbox_fixed: type fixed, parent hand_yaw_motor_link, child hand_yaw_gearbox_link, origin xyz=0 0 0
- added joint hand_yaw_motor_fixed: type fixed, parent hand_adapter_link, child hand_yaw_motor_link, origin xyz=0.03 0 0
- added joint knuckle_spread_L_gearbox_fixed: type fixed, parent knuckle_spread_L_motor_link, child knuckle_spread_L_gearbox_link, origin xyz=0 0 0
- added joint knuckle_spread_L_motor_fixed: type fixed, parent hand_palm_link, child knuckle_spread_L_motor_link, origin xyz=0.105 -0.03 0
- added joint knuckle_spread_R_gearbox_fixed: type fixed, parent knuckle_spread_R_motor_link, child knuckle_spread_R_gearbox_link, origin xyz=0 0 0
- added joint knuckle_spread_R_motor_fixed: type fixed, parent hand_palm_link, child knuckle_spread_R_motor_link, origin xyz=0.105 0.03 0
- joint finger_L_prismatic_joint: origin xyz=0.012 -0.005 0.015 -> xyz=0 0 0; parent hand_knuckle_l_link -> finger_L_gearbox_link
- joint finger_R_prismatic_joint: origin xyz=0.012 0.005 0.015 -> xyz=0 0 0; parent hand_knuckle_r_link -> finger_R_gearbox_link
- joint hand_pitch_joint: origin xyz=0.025 0 0 -> xyz=0 0 0; parent hand_yaw_link -> hand_pitch_gearbox_link
- joint hand_roll_joint: origin xyz=0.025 0 0 -> xyz=0 0 0; parent hand_pitch_link -> hand_roll_gearbox_link
- joint hand_yaw_joint: origin xyz=0.03 0 0 -> xyz=0 0 0; parent hand_adapter_link -> hand_yaw_gearbox_link
- joint knuckle_spread_L_joint: origin xyz=0.105 -0.03 0 -> xyz=0 0 0; parent hand_palm_link -> knuckle_spread_L_gearbox_link
- joint knuckle_spread_R_joint: origin xyz=0.105 0.03 0 -> xyz=0 0 0; parent hand_palm_link -> knuckle_spread_R_gearbox_link

File: freecad_hand_7dof/urdf/hand_7dof.urdf (robot description, URDF)
Before this commit: robot hand_7dof, 8 links, 8 joints
Links:
- added link finger_L_gearbox_link, mass 0.060; collision cylinder length=0.025 radius=0.014; visual cylinder length=0.025 radius=0.014
- added link finger_L_motor_link, mass 0.040; collision cylinder length=0.030 radius=0.010; visual cylinder length=0.030 radius=0.010
- added link finger_R_gearbox_link, mass 0.060; collision cylinder length=0.025 radius=0.014; visual cylinder length=0.025 radius=0.014
- added link finger_R_motor_link, mass 0.040; collision cylinder length=0.030 radius=0.010; visual cylinder length=0.030 radius=0.010
- added link hand_pitch_gearbox_link, mass 0.200; collision cylinder length=0.040 radius=0.025; visual cylinder length=0.040 radius=0.025
- added link hand_pitch_motor_link, mass 0.150; collision cylinder length=0.030 radius=0.0225; visual cylinder length=0.030 radius=0.0225
- added link hand_roll_gearbox_link, mass 0.120; collision cylinder length=0.035 radius=0.019; visual cylinder length=0.035 radius=0.019
- added link hand_roll_motor_link, mass 0.080; collision cylinder length=0.040 radius=0.016; visual cylinder length=0.040 radius=0.016
- added link hand_yaw_gearbox_link, mass 0.200; collision cylinder length=0.040 radius=0.025; visual cylinder length=0.040 radius=0.025
- added link hand_yaw_motor_link, mass 0.150; collision cylinder length=0.030 radius=0.0225; visual cylinder length=0.030 radius=0.0225
- added link knuckle_spread_L_gearbox_link, mass 0.080; collision cylinder length=0.025 radius=0.014; visual cylinder length=0.025 radius=0.014
- added link knuckle_spread_L_motor_link, mass 0.050; collision cylinder length=0.030 radius=0.011; visual cylinder length=0.030 radius=0.011
- added link knuckle_spread_R_gearbox_link, mass 0.080; collision cylinder length=0.025 radius=0.014; visual cylinder length=0.025 radius=0.014
- added link knuckle_spread_R_motor_link, mass 0.050; collision cylinder length=0.030 radius=0.011; visual cylinder length=0.030 radius=0.011
Joints:
- added joint finger_L_gearbox_fixed: type fixed, parent finger_L_motor_link, child finger_L_gearbox_link, origin xyz=0 0 0
- added joint finger_L_motor_fixed: type fixed, parent hand_knuckle_l_link, child finger_L_motor_link, origin xyz=0.012 -0.005 0.015
- added joint finger_R_gearbox_fixed: type fixed, parent finger_R_motor_link, child finger_R_gearbox_link, origin xyz=0 0 0
- added joint finger_R_motor_fixed: type fixed, parent hand_knuckle_r_link, child finger_R_motor_link, origin xyz=0.012 0.005 0.015
- added joint hand_pitch_gearbox_fixed: type fixed, parent hand_pitch_motor_link, child hand_pitch_gearbox_link, origin xyz=0 0 0
- added joint hand_pitch_motor_fixed: type fixed, parent hand_yaw_link, child hand_pitch_motor_link, origin xyz=0.025 0 0
- added joint hand_roll_gearbox_fixed: type fixed, parent hand_roll_motor_link, child hand_roll_gearbox_link, origin xyz=0 0 0
- added joint hand_roll_motor_fixed: type fixed, parent hand_pitch_link, child hand_roll_motor_link, origin xyz=0.025 0 0
- added joint hand_yaw_gearbox_fixed: type fixed, parent hand_yaw_motor_link, child hand_yaw_gearbox_link, origin xyz=0 0 0
- added joint hand_yaw_motor_fixed: type fixed, parent hand_adapter_link, child hand_yaw_motor_link, origin xyz=0.03 0 0
- added joint knuckle_spread_L_gearbox_fixed: type fixed, parent knuckle_spread_L_motor_link, child knuckle_spread_L_gearbox_link, origin xyz=0 0 0
- added joint knuckle_spread_L_motor_fixed: type fixed, parent hand_palm_link, child knuckle_spread_L_motor_link, origin xyz=0.105 -0.03 0
- added joint knuckle_spread_R_gearbox_fixed: type fixed, parent knuckle_spread_R_motor_link, child knuckle_spread_R_gearbox_link, origin xyz=0 0 0
- added joint knuckle_spread_R_motor_fixed: type fixed, parent hand_palm_link, child knuckle_spread_R_motor_link, origin xyz=0.105 0.03 0
- joint finger_L_prismatic_joint: origin xyz=0.012 -0.005 0.015 -> xyz=0 0 0; parent hand_knuckle_l_link -> finger_L_gearbox_link
- joint finger_R_prismatic_joint: origin xyz=0.012 0.005 0.015 -> xyz=0 0 0; parent hand_knuckle_r_link -> finger_R_gearbox_link
- joint hand_pitch_joint: origin xyz=0.025 0 0 -> xyz=0 0 0; parent hand_yaw_link -> hand_pitch_gearbox_link
- joint hand_roll_joint: origin xyz=0.025 0 0 -> xyz=0 0 0; parent hand_pitch_link -> hand_roll_gearbox_link
- joint hand_yaw_joint: origin xyz=0.03 0 0 -> xyz=0 0 0; parent hand_adapter_link -> hand_yaw_gearbox_link
- joint knuckle_spread_L_joint: origin xyz=0.105 -0.03 0 -> xyz=0 0 0; parent hand_palm_link -> knuckle_spread_L_gearbox_link
- joint knuckle_spread_R_joint: origin xyz=0.105 0.03 0 -> xyz=0 0 0; parent hand_palm_link -> knuckle_spread_R_gearbox_link
