Commit message: feat: V2 anthropomorphic 5-finger hand with phalanges, mimic joints, STS3215 pod
- build_v2_hand.py: numpy mesh generator for 5-finger hand (32 STLs)
  - Palm plate 130×70×18mm with 5 finger bosses + cable ridge
  - Thumb: CMC base + proximal + distal phalanges (hemisphere domes)
  - 4 fingers: knuckle bracket (683ZZ pocket) + proximal + middle + distal
  - Each phalanx has spherical joint bosses for realistic DOF
- hand_7dof.urdf: 7 actuated + 7 mimic joints (14 total, 30 links)
  - A1 thumb CMC opposition (Z ±45°), A2 thumb MCP flexion (Y 0..90°)
  - A3-A6 index/middle/ring/little MCP flexion (Y 0..90°)
  - PIP mimic at 0.85× MCP, DIP mimic at 0.6× PIP per finger
  - Forearm pod link (0.08×0.028m cylinder) houses all 7 STS3215 servos
  - PETG-computed inertias (1.25 g/cm³ density), ~380g hand mass
- assemble_full_urdf.py: regenerated for V2 kinematics
- ros2_control.yaml: updated to 7 hand joints
- README: documented V2 changes, kinematics, control examples

File: freecad_hand_7dof/urdf/fetch_7dof_with_hand.urdf (robot description, URDF)
Before this commit: robot fetch_7dof, 31 links, 30 joints
Links:
- removed link finger_L_gearbox_link
- removed link finger_L_motor_link
- removed link finger_R_gearbox_link
- removed link finger_R_motor_link
- removed link hand_finger_l_link
- removed link hand_finger_r_link
- removed link hand_knuckle_l_link
- removed link hand_knuckle_r_link
- removed link hand_pitch_gearbox_link
- removed link hand_pitch_link
- removed link hand_pitch_motor_link
- removed link hand_roll_gearbox_link
- removed link hand_roll_motor_link
- removed link hand_yaw_gearbox_link
- removed link hand_yaw_link
- removed link hand_yaw_motor_link
- removed link knuckle_spread_L_gearbox_link
- removed link knuckle_spread_L_motor_link
- removed link knuckle_spread_R_gearbox_link
- removed link knuckle_spread_R_motor_link
- added link hand_pod_link, mass 0.450; collision cylinder length=0.080 radius=0.028; visual cylinder length=0.080 radius=0.028
- added link index_D_link, mass 0.001; collision mesh filename=package://freecad_hand_7dof/meshes/index_D_link.stl scale=0.001 0.001 0.001; visual mesh filename=package://freecad_hand_7dof/meshes/index_D_link.stl scale=0.001 0.001 0.001
- added link index_K_link, mass 0.002; collision mesh filename=package://freecad_hand_7dof/meshes/index_K_link.stl scale=0.001 0.001 0.001; visual mesh filename=package://freecad_hand_7dof/meshes/index_K_link.stl scale=0.001 0.001 0.001
- added link index_M_link, mass 0.002; collision mesh filename=package://freecad_hand_7dof/meshes/index_M_link.stl scale=0.001 0.001 0.001; visual mesh filename=package://freecad_hand_7dof/meshes/index_M_link.stl scale=0.001 0.001 0.001
- added link index_P_link, mass 0.003; collision mesh filename=package://freecad_hand_7dof/meshes/index_P_link.stl scale=0.001 0.001 0.001; visual mesh filename=package://freecad_hand_7dof/meshes/index_P_link.stl scale=0.001 0.001 0.001
- added link little_D_link, mass 0.001; collision mesh filename=package://freecad_hand_7dof/meshes/little_D_link.stl scale=0.001 0.001 0.001; visual mesh filename=package://freecad_hand_7dof/meshes/little_D_link.stl scale=0.001 0.001 0.001
- added link little_K_link, mass 0.002; collision mesh filename=package://freecad_hand_7dof/meshes/little_K_link.stl scale=0.001 0.001 0.001; visual mesh filename=package://freecad_hand_7dof/meshes/little_K_link.stl scale=0.001 0.001 0.001
- added link little_M_link, mass 0.002; collision mesh filename=package://freecad_hand_7dof/meshes/little_M_link.stl scale=0.001 0.001 0.001; visual mesh filename=package://freecad_hand_7dof/meshes/little_M_link.stl scale=0.001 0.001 0.001
- added link little_P_link, mass 0.003; collision mesh filename=package://freecad_hand_7dof/meshes/little_P_link.stl scale=0.001 0.001 0.001; visual mesh filename=package://freecad_hand_7dof/meshes/little_P_link.stl scale=0.001 0.001 0.001
- added link middle_D_link, mass 0.001; collision mesh filename=package://freecad_hand_7dof/meshes/middle_D_link.stl scale=0.001 0.001 0.001; visual mesh filename=package://freecad_hand_7dof/meshes/middle_D_link.stl scale=0.001 0.001 0.001
- added link middle_K_link, mass 0.002; collision mesh filename=package://freecad_hand_7dof/meshes/middle_K_link.stl scale=0.001 0.001 0.001; visual mesh filename=package://freecad_hand_7dof/meshes/middle_K_link.stl scale=0.001 0.001 0.001
- added link middle_M_link, mass 0.002; collision mesh filename=package://freecad_hand_7dof/meshes/middle_M_link.stl scale=0.001 0.001 0.001; visual mesh filename=package://freecad_hand_7dof/meshes/middle_M_link.stl scale=0.001 0.001 0.001
- added link middle_P_link, mass 0.003; collision mesh filename=package://freecad_hand_7dof/meshes/middle_P_link.stl scale=0.001 0.001 0.001; visual mesh filename=package://freecad_hand_7dof/meshes/middle_P_link.stl scale=0.001 0.001 0.001
- added link ring_D_link, mass 0.001; collision mesh filename=package://freecad_hand_7dof/meshes/ring_D_link.stl scale=0.001 0.001 0.001; visual mesh filename=package://freecad_hand_7dof/meshes/ring_D_link.stl scale=0.001 0.001 0.001
- added link ring_K_link, mass 0.002; collision mesh filename=package://freecad_hand_7dof/meshes/ring_K_link.stl scale=0.001 0.001 0.001; visual mesh filename=package://freecad_hand_7dof/meshes/ring_K_link.stl scale=0.001 0.001 0.001
- added link ring_M_link, mass 0.002; collision mesh filename=package://freecad_hand_7dof/meshes/ring_M_link.stl scale=0.001 0.001 0.001; visual mesh filename=package://freecad_hand_7dof/meshes/ring_M_link.stl scale=0.001 0.001 0.001
- added link ring_P_link, mass 0.003; collision mesh filename=package://freecad_hand_7dof/meshes/ring_P_link.stl scale=0.001 0.001 0.001; visual mesh filename=package://freecad_hand_7dof/meshes/ring_P_link.stl scale=0.001 0.001 0.001
- added link thumb_D_link, mass 0.003; collision mesh filename=package://freecad_hand_7dof/meshes/thumb_D_link.stl scale=0.001 0.001 0.001; visual mesh filename=package://freecad_hand_7dof/meshes/thumb_D_link.stl scale=0.001 0.001 0.001
- added link thumb_P_link, mass 0.005; collision mesh filename=package://freecad_hand_7dof/meshes/thumb_P_link.stl scale=0.001 0.001 0.001; visual mesh filename=package://freecad_hand_7dof/meshes/thumb_P_link.stl scale=0.001 0.001 0.001
- added link thumb_base_link, mass 0.005; collision mesh filename=package://freecad_hand_7dof/meshes/thumb_base_link.stl scale=0.001 0.001 0.001; visual mesh filename=package://freecad_hand_7dof/meshes/thumb_base_link.stl scale=0.001 0.001 0.001
- link hand_adapter_link: mass 0.12 -> 0.196; geometry collision mesh filename=package://freecad_hand_7dof/meshes/hand_adapter_link.stl scale=0.001 0.001 0.001; visual mesh filename=package://freecad_hand_7dof/meshes/hand_adapter_link.stl scale=0.001 0.001 0.001
- link hand_palm_link: mass 0.25 -> 0.455; geometry collision mesh filename=package://freecad_hand_7dof/meshes/hand_palm_link.stl scale=0.001 0.001 0.001; visual mesh filename=package://freecad_hand_7dof/meshes/hand_palm_link.stl scale=0.001 0.001 0.001
Joints:
- removed joint finger_L_gearbox_fixed
- removed joint finger_L_motor_fixed
- removed joint finger_L_prismatic_joint
- removed joint finger_R_gearbox_fixed
- removed joint finger_R_motor_fixed
- removed joint finger_R_prismatic_joint
- removed joint hand_pitch_gearbox_fixed
- removed joint hand_pitch_joint
- removed joint hand_pitch_motor_fixed
- removed joint hand_roll_gearbox_fixed
- removed joint hand_roll_joint
- removed joint hand_roll_motor_fixed
- removed joint hand_yaw_gearbox_fixed
- removed joint hand_yaw_joint
- removed joint hand_yaw_motor_fixed
- removed joint knuckle_spread_L_gearbox_fixed
- removed joint knuckle_spread_L_joint
- removed joint knuckle_spread_L_motor_fixed
- removed joint knuckle_spread_R_gearbox_fixed
- removed joint knuckle_spread_R_joint
- removed joint knuckle_spread_R_motor_fixed
- added joint index_dip_joint: type revolute, parent index_M_link, child index_D_link, origin xyz=0.020 0 0, axis 0 1 0, limit lower=0.0 upper=0.959 effort=1.0 velocity=2.0, mimic joint=index_pic_joint multiplier=0.6 offset=0.0
- added joint index_knuckle_fixed: type fixed, parent hand_palm_link, child index_K_link, origin xyz=0.120 -0.015 0.027
- added joint index_mcp_joint: type revolute, parent index_K_link, child index_P_link, origin xyz=0 0 0, axis 0 1 0, limit lower=0.0 upper=1.5708 effort=2.5 velocity=2.0
- added joint index_pic_joint: type revolute, parent index_P_link, child index_M_link, origin xyz=0.026 0 0, axis 0 1 0, limit lower=0.0 upper=1.309 effort=1.5 velocity=2.0, mimic joint=index_mcp_joint multiplier=0.85 offset=0.0
- added joint little_dip_joint: type revolute, parent little_M_link, child little_D_link, origin xyz=0.016 0 0, axis 0 1 0, limit lower=0.0 upper=0.959 effort=1.0 velocity=2.0, mimic joint=little_pic_joint multiplier=0.6 offset=0.0
- added joint little_knuckle_fixed: type fixed, parent hand_palm_link, child little_K_link, origin xyz=0.120 0.030 0.027
- added joint little_mcp_joint: type revolute, parent little_K_link, child little_P_link, origin xyz=0 0 0, axis 0 1 0, limit lower=0.0 upper=1.5708 effort=2.5 velocity=2.0
- added joint little_pic_joint: type revolute, parent little_P_link, child little_M_link, origin xyz=0.022 0 0, axis 0 1 0, limit lower=0.0 upper=1.309 effort=1.5 velocity=2.0, mimic joint=little_mcp_joint multiplier=0.85 offset=0.0
- added joint middle_dip_joint: type revolute, parent middle_M_link, child middle_D_link, origin xyz=0.022 0 0, axis 0 1 0, limit lower=0.0 upper=0.959 effort=1.0 velocity=2.0, mimic joint=middle_pic_joint multiplier=0.6 offset=0.0
- added joint middle_knuckle_fixed: type fixed, parent hand_palm_link, child middle_K_link, origin xyz=0.120 0.000 0.027
- added joint middle_mcp_joint: type revolute, parent middle_K_link, child middle_P_link, origin xyz=0 0 0, axis 0 1 0, limit lower=0.0 upper=1.5708 effort=2.5 velocity=2.0
- added joint middle_pic_joint: type revolute, parent middle_P_link, child middle_M_link, origin xyz=0.028 0 0, axis 0 1 0, limit lower=0.0 upper=1.309 effort=1.5 velocity=2.0, mimic joint=middle_mcp_joint multiplier=0.85 offset=0.0
- added joint palm_fixed: type fixed, parent hand_adapter_link, child hand_palm_link, origin xyz=0.065 0 0
- added joint pod_fixed: type fixed, parent hand_adapter_link, child hand_pod_link, origin xyz=-0.055 0 0 rpy=0 0 0
- added joint ring_dip_joint: type revolute, parent ring_M_link, child ring_D_link, origin xyz=0.020 0 0, axis 0 1 0, limit lower=0.0 upper=0.959 effort=1.0 velocity=2.0, mimic joint=ring_pic_joint multiplier=0.6 offset=0.0
- added joint ring_knuckle_fixed: type fixed, parent hand_palm_link, child ring_K_link, origin xyz=0.120 0.015 0.027
- added joint ring_mcp_joint: type revolute, parent ring_K_link, child ring_P_link, origin xyz=0 0 0, axis 0 1 0, limit lower=0.0 upper=1.5708 effort=2.5 velocity=2.0
- added joint ring_pic_joint: type revolute, parent ring_P_link, child ring_M_link, origin xyz=0.026 0 0, axis 0 1 0, limit lower=0.0 upper=1.309 effort=1.5 velocity=2.0, mimic joint=ring_mcp_joint multiplier=0.85 offset=0.0
- added joint thumb_base_fixed: type fixed, parent hand_palm_link, child thumb_base_link, origin xyz=0.115 -0.032 0.018 rpy=0 0 0.3
- added joint thumb_cmcmc_joint: type revolute, parent thumb_base_link, child thumb_P_link, origin xyz=0.012 0.011 0.008 rpy=0 0 0, axis 0 0 1, limit lower=-0.7854 upper=0.7854 effort=5.0 velocity=2.0
- added joint thumb_mcp_joint: type revolute, parent thumb_P_link, child thumb_D_link, origin xyz=0.022 0 0 rpy=0 0 0, axis 0 1 0, limit lower=0.0 upper=1.5708 effort=3.0 velocity=2.0

File: freecad_hand_7dof/urdf/hand_7dof.urdf (robot description, URDF)
Before this commit: robot hand_7dof, 22 links, 22 joints
Links:
- removed link finger_L_gearbox_link
- removed link finger_L_motor_link
- removed link finger_R_gearbox_link
- removed link finger_R_motor_link
- removed link hand_finger_l_link
- removed link hand_finger_r_link
- removed link hand_knuckle_l_link
- removed link hand_knuckle_r_link
- removed link hand_pitch_gearbox_link
- removed link hand_pitch_link
- removed link hand_pitch_motor_link
- removed link hand_roll_gearbox_link
- removed link hand_roll_motor_link
- removed link hand_yaw_gearbox_link
- removed link hand_yaw_link
- removed link hand_yaw_motor_link
- removed link knuckle_spread_L_gearbox_link
- removed link knuckle_spread_L_motor_link
- removed link knuckle_spread_R_gearbox_link
- removed link knuckle_spread_R_motor_link
- added link hand_pod_link, mass 0.450; collision cylinder length=0.080 radius=0.028; visual cylinder length=0.080 radius=0.028
- added link index_D_link, mass 0.001; collision mesh filename=package://freecad_hand_7dof/meshes/index_D_link.stl scale=0.001 0.001 0.001; visual mesh filename=package://freecad_hand_7dof/meshes/index_D_link.stl scale=0.001 0.001 0.001
- added link index_K_link, mass 0.002; collision mesh filename=package://freecad_hand_7dof/meshes/index_K_link.stl scale=0.001 0.001 0.001; visual mesh filename=package://freecad_hand_7dof/meshes/index_K_link.stl scale=0.001 0.001 0.001
- added link index_M_link, mass 0.002; collision mesh filename=package://freecad_hand_7dof/meshes/index_M_link.stl scale=0.001 0.001 0.001; visual mesh filename=package://freecad_hand_7dof/meshes/index_M_link.stl scale=0.001 0.001 0.001
- added link index_P_link, mass 0.003; collision mesh filename=package://freecad_hand_7dof/meshes/index_P_link.stl scale=0.001 0.001 0.001; visual mesh filename=package://freecad_hand_7dof/meshes/index_P_link.stl scale=0.001 0.001 0.001
- added link little_D_link, mass 0.001; collision mesh filename=package://freecad_hand_7dof/meshes/little_D_link.stl scale=0.001 0.001 0.001; visual mesh filename=package://freecad_hand_7dof/meshes/little_D_link.stl scale=0.001 0.001 0.001
- added link little_K_link, mass 0.002; collision mesh filename=package://freecad_hand_7dof/meshes/little_K_link.stl scale=0.001 0.001 0.001; visual mesh filename=package://freecad_hand_7dof/meshes/little_K_link.stl scale=0.001 0.001 0.001
- added link little_M_link, mass 0.002; collision mesh filename=package://freecad_hand_7dof/meshes/little_M_link.stl scale=0.001 0.001 0.001; visual mesh filename=package://freecad_hand_7dof/meshes/little_M_link.stl scale=0.001 0.001 0.001
- added link little_P_link, mass 0.003; collision mesh filename=package://freecad_hand_7dof/meshes/little_P_link.stl scale=0.001 0.001 0.001; visual mesh filename=package://freecad_hand_7dof/meshes/little_P_link.stl scale=0.001 0.001 0.001
- added link middle_D_link, mass 0.001; collision mesh filename=package://freecad_hand_7dof/meshes/middle_D_link.stl scale=0.001 0.001 0.001; visual mesh filename=package://freecad_hand_7dof/meshes/middle_D_link.stl scale=0.001 0.001 0.001
- added link middle_K_link, mass 0.002; collision mesh filename=package://freecad_hand_7dof/meshes/middle_K_link.stl scale=0.001 0.001 0.001; visual mesh filename=package://freecad_hand_7dof/meshes/middle_K_link.stl scale=0.001 0.001 0.001
- added link middle_M_link, mass 0.002; collision mesh filename=package://freecad_hand_7dof/meshes/middle_M_link.stl scale=0.001 0.001 0.001; visual mesh filename=package://freecad_hand_7dof/meshes/middle_M_link.stl scale=0.001 0.001 0.001
- added link middle_P_link, mass 0.003; collision mesh filename=package://freecad_hand_7dof/meshes/middle_P_link.stl scale=0.001 0.001 0.001; visual mesh filename=package://freecad_hand_7dof/meshes/middle_P_link.stl scale=0.001 0.001 0.001
- added link ring_D_link, mass 0.001; collision mesh filename=package://freecad_hand_7dof/meshes/ring_D_link.stl scale=0.001 0.001 0.001; visual mesh filename=package://freecad_hand_7dof/meshes/ring_D_link.stl scale=0.001 0.001 0.001
- added link ring_K_link, mass 0.002; collision mesh filename=package://freecad_hand_7dof/meshes/ring_K_link.stl scale=0.001 0.001 0.001; visual mesh filename=package://freecad_hand_7dof/meshes/ring_K_link.stl scale=0.001 0.001 0.001
- added link ring_M_link, mass 0.002; collision mesh filename=package://freecad_hand_7dof/meshes/ring_M_link.stl scale=0.001 0.001 0.001; visual mesh filename=package://freecad_hand_7dof/meshes/ring_M_link.stl scale=0.001 0.001 0.001
- added link ring_P_link, mass 0.003; collision mesh filename=package://freecad_hand_7dof/meshes/ring_P_link.stl scale=0.001 0.001 0.001; visual mesh filename=package://freecad_hand_7dof/meshes/ring_P_link.stl scale=0.001 0.001 0.001
- added link thumb_D_link, mass 0.003; collision mesh filename=package://freecad_hand_7dof/meshes/thumb_D_link.stl scale=0.001 0.001 0.001; visual mesh filename=package://freecad_hand_7dof/meshes/thumb_D_link.stl scale=0.001 0.001 0.001
- added link thumb_P_link, mass 0.005; collision mesh filename=package://freecad_hand_7dof/meshes/thumb_P_link.stl scale=0.001 0.001 0.001; visual mesh filename=package://freecad_hand_7dof/meshes/thumb_P_link.stl scale=0.001 0.001 0.001
- added link thumb_base_link, mass 0.005; collision mesh filename=package://freecad_hand_7dof/meshes/thumb_base_link.stl scale=0.001 0.001 0.001; visual mesh filename=package://freecad_hand_7dof/meshes/thumb_base_link.stl scale=0.001 0.001 0.001
- link hand_adapter_link: mass 0.12 -> 0.196; geometry collision mesh filename=package://freecad_hand_7dof/meshes/hand_adapter_link.stl scale=0.001 0.001 0.001; visual mesh filename=package://freecad_hand_7dof/meshes/hand_adapter_link.stl scale=0.001 0.001 0.001
- link hand_palm_link: mass 0.25 -> 0.455; geometry collision mesh filename=package://freecad_hand_7dof/meshes/hand_palm_link.stl scale=0.001 0.001 0.001; visual mesh filename=package://freecad_hand_7dof/meshes/hand_palm_link.stl scale=0.001 0.001 0.001
Joints:
- removed joint finger_L_gearbox_fixed
- removed joint finger_L_motor_fixed
- removed joint finger_L_prismatic_joint
- removed joint finger_R_gearbox_fixed
- removed joint finger_R_motor_fixed
- removed joint finger_R_prismatic_joint
- removed joint hand_pitch_gearbox_fixed
- removed joint hand_pitch_joint
- removed joint hand_pitch_motor_fixed
- removed joint hand_roll_gearbox_fixed
- removed joint hand_roll_joint
- removed joint hand_roll_motor_fixed
- removed joint hand_yaw_gearbox_fixed
- removed joint hand_yaw_joint
- removed joint hand_yaw_motor_fixed
- removed joint knuckle_spread_L_gearbox_fixed
- removed joint knuckle_spread_L_joint
- removed joint knuckle_spread_L_motor_fixed
- removed joint knuckle_spread_R_gearbox_fixed
- removed joint knuckle_spread_R_joint
- removed joint knuckle_spread_R_motor_fixed
- added joint index_dip_joint: type revolute, parent index_M_link, child index_D_link, origin xyz=0.020 0 0, axis 0 1 0, limit lower=0.0 upper=0.959 effort=1.0 velocity=2.0, mimic joint=index_pic_joint multiplier=0.6 offset=0.0
- added joint index_knuckle_fixed: type fixed, parent hand_palm_link, child index_K_link, origin xyz=0.120 -0.015 0.027
- added joint index_mcp_joint: type revolute, parent index_K_link, child index_P_link, origin xyz=0 0 0, axis 0 1 0, limit lower=0.0 upper=1.5708 effort=2.5 velocity=2.0
- added joint index_pic_joint: type revolute, parent index_P_link, child index_M_link, origin xyz=0.026 0 0, axis 0 1 0, limit lower=0.0 upper=1.309 effort=1.5 velocity=2.0, mimic joint=index_mcp_joint multiplier=0.85 offset=0.0
- added joint little_dip_joint: type revolute, parent little_M_link, child little_D_link, origin xyz=0.016 0 0, axis 0 1 0, limit lower=0.0 upper=0.959 effort=1.0 velocity=2.0, mimic joint=little_pic_joint multiplier=0.6 offset=0.0
- added joint little_knuckle_fixed: type fixed, parent hand_palm_link, child little_K_link, origin xyz=0.120 0.030 0.027
- added joint little_mcp_joint: type revolute, parent little_K_link, child little_P_link, origin xyz=0 0 0, axis 0 1 0, limit lower=0.0 upper=1.5708 effort=2.5 velocity=2.0
- added joint little_pic_joint: type revolute, parent little_P_link, child little_M_link, origin xyz=0.022 0 0, axis 0 1 0, limit lower=0.0 upper=1.309 effort=1.5 velocity=2.0, mimic joint=little_mcp_joint multiplier=0.85 offset=0.0
- added joint middle_dip_joint: type revolute, parent middle_M_link, child middle_D_link, origin xyz=0.022 0 0, axis 0 1 0, limit lower=0.0 upper=0.959 effort=1.0 velocity=2.0, mimic joint=middle_pic_joint multiplier=0.6 offset=0.0
- added joint middle_knuckle_fixed: type fixed, parent hand_palm_link, child middle_K_link, origin xyz=0.120 0.000 0.027
- added joint middle_mcp_joint: type revolute, parent middle_K_link, child middle_P_link, origin xyz=0 0 0, axis 0 1 0, limit lower=0.0 upper=1.5708 effort=2.5 velocity=2.0
- added joint middle_pic_joint: type revolute, parent middle_P_link, child middle_M_link, origin xyz=0.028 0 0, axis 0 1 0, limit lower=0.0 upper=1.309 effort=1.5 velocity=2.0, mimic joint=middle_mcp_joint multiplier=0.85 offset=0.0
- added joint palm_fixed: type fixed, parent hand_adapter_link, child hand_palm_link, origin xyz=0.065 0 0
- added joint pod_fixed: type fixed, parent hand_adapter_link, child hand_pod_link, origin xyz=-0.055 0 0 rpy=0 0 0
- added joint ring_dip_joint: type revolute, parent ring_M_link, child ring_D_link, origin xyz=0.020 0 0, axis 0 1 0, limit lower=0.0 upper=0.959 effort=1.0 velocity=2.0, mimic joint=ring_pic_joint multiplier=0.6 offset=0.0
- added joint ring_knuckle_fixed: type fixed, parent hand_palm_link, child ring_K_link, origin xyz=0.120 0.015 0.027
- added joint ring_mcp_joint: type revolute, parent ring_K_link, child ring_P_link, origin xyz=0 0 0, axis 0 1 0, limit lower=0.0 upper=1.5708 effort=2.5 velocity=2.0
- added joint ring_pic_joint: type revolute, parent ring_P_link, child ring_M_link, origin xyz=0.026 0 0, axis 0 1 0, limit lower=0.0 upper=1.309 effort=1.5 velocity=2.0, mimic joint=ring_mcp_joint multiplier=0.85 offset=0.0
- added joint thumb_base_fixed: type fixed, parent hand_palm_link, child thumb_base_link, origin xyz=0.115 -0.032 0.018 rpy=0 0 0.3
- added joint thumb_cmcmc_joint: type revolute, parent thumb_base_link, child thumb_P_link, origin xyz=0.012 0.011 0.008 rpy=0 0 0, axis 0 0 1, limit lower=-0.7854 upper=0.7854 effort=5.0 velocity=2.0
- added joint thumb_mcp_joint: type revolute, parent thumb_P_link, child thumb_D_link, origin xyz=0.022 0 0 rpy=0 0 0, axis 0 1 0, limit lower=0.0 upper=1.5708 effort=3.0 velocity=2.0
