Commit message: feat: build 7-DOF serial arm from scratch with proper solid geometry
- arm_7dof.FCStd: FreeCAD document with 16 Part::Feature solids
  (BasePlate + 7 Servo bodies + 7 Horns + EndEffector)
  - No triangle meshes (.bms), all parametric B-Rep solids
  - Proper transform chain: each servo horn attaches to previous link

- arm_7dof.urdf: 7-DOF serial manipulator URDF
  - J1-J7: Z/Y/Z/Y/Z/Y/Z axes, ±180° limits, 5Nm effort
  - STS3215 servo specs (0.135kg per link, cylinder visual)
  - SimpleTransmission with 10:1 reduction

- build_arm.py: FreeCAD script to regenerate FCStd

Total reach: ~430mm from base to end effector

File: freecad_hand_7dof/arm_7dof.urdf (robot description, URDF)
Before this commit: robot arm_7dof, 9 links, 8 joints
Links:
- link link_0: geometry collision cylinder length=0.045 radius=0.02; visual cylinder length=0.045 radius=0.02
- link link_1: geometry collision cylinder length=0.045 radius=0.02; visual cylinder length=0.045 radius=0.02
- link link_2: geometry collision cylinder length=0.045 radius=0.02; visual cylinder length=0.045 radius=0.02
- link link_3: geometry collision cylinder length=0.045 radius=0.02; visual cylinder length=0.045 radius=0.02
- link link_4: geometry collision cylinder length=0.045 radius=0.02; visual cylinder length=0.045 radius=0.02
- link link_5: geometry collision cylinder length=0.045 radius=0.02; visual cylinder length=0.045 radius=0.02
- link link_6: geometry collision cylinder length=0.045 radius=0.02; visual cylinder length=0.045 radius=0.02
Joints:
- removed joint joint_0
- removed joint joint_1
- removed joint joint_2
- removed joint joint_3
- removed joint joint_4
- removed joint joint_5
- removed joint joint_6
- removed joint joint_7
- added joint joint_J1: type revolute, parent base_link, child link_0, origin xyz=0 0 0.045 rpy=0 0 0, axis 0 0 1, limit 
- added joint joint_J2: type revolute, parent link_0, child link_1, origin xyz=0 0 0.045 rpy=0 0 0, axis 0 1 0, limit 
- added joint joint_J3: type revolute, parent link_1, child link_2, origin xyz=0 0 0.045 rpy=0 0 0, axis 0 0 1, limit 
- added joint joint_J4: type revolute, parent link_2, child link_3, origin xyz=0 0 0.045 rpy=0 0 0, axis 0 1 0, limit 
- added joint joint_J5: type revolute, parent link_3, child link_4, origin xyz=0 0 0.045 rpy=0 0 0, axis 0 0 1, limit 
- added joint joint_J6: type revolute, parent link_4, child link_5, origin xyz=0 0 0.045 rpy=0 0 0, axis 0 1 0, limit 
- added joint joint_J7: type revolute, parent link_5, child link_6, origin xyz=0 0 0.045 rpy=0 0 0, axis 0 0 1, limit 
- added joint joint_end: type fixed, parent link_6, child end_effector, origin xyz=0 0 0.02 rpy=0 0 0
